Commit message: Add exercise

File: sample_robot_bringup/launch/single_rrbot.urdf (robot description, URDF)
Before this commit: robot single_rrbot, 5 links, 4 joints
Links:
- added link single_rrbot_link5
Joints:
- added joint single_rrbot_joint4: type prismatic, parent single_rrbot_link4, child single_rrbot_link5, origin xyz=0 0 -0.1 rpy=0 0 0, axis 0 0 1, limit lower=0.0 upper=-1.0 effort=30.0 velocity=1.0
- joint single_rrbot_joint1: limit lower=0.0 upper=1.0 effort=30.0 velocity=1.0 -> (none); origin xyz=0 0.1 0.5 rpy=0 0 0 -> xyz=0 0 1 rpy=0 0 0; type prismatic -> continuous
- joint single_rrbot_joint2: axis 0 1 0 -> 0 0 1; origin xyz=0 0.1 1.0 rpy=0 0 0 -> xyz=1 0 0 rpy=0 0 0
- joint single_rrbot_joint3: axis 0 1 0 -> 0 0 1; origin xyz=0 0.1 0.9 rpy=0 0 0 -> xyz=0 1 0 rpy=0 0 0
